File: signal.kicad_sch (KiCad schematic)
At the start: 130 parts, among them Q1 MMBFJ202, Q10 BC848C, Q11 BC848C, Q12 BC848C, Q13 BC848C, Q2 MMBFJ202, Q3 MMBFJ202, Q4 MMBFJ202, Q5 BC848C, Q6 LS844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

Commit message: start of PCB re-route
Parts:
- SW2: footprint (none) -> bca-footprints:Pin_Header_Straight_1x06_Pitch2.54mm

Commit message: first draft of PCB
Connections:
- net ccs0: no longer SW2.3 (C)
- net at C35.2, C36.1, C37.2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: now also U3.7; no longer U3.1
- net at C21.2, R24.2, R25.1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: now also U3.3 (+); no longer U3.5 (+)
- net at Q1.2 (S), R5.1, R6.1: now also SW2.3 (C)
- net at R42.2: now also U3.6 (-); no longer U3.2 (-)
- net at R43.2: now also U3.5 (+); no longer U3.3 (+)
- net at C26.1, R31.2, RV2.3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: now also U3.2 (-); no longer U3.6 (-)
- net at C26.2, C27.2, R31.1: now also U3.1; no longer U3.7
Changed lines of the file:
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@@
   (junction (at 44.45 40.64) (diameter 0) (color 0 0 0 0)
   )
-  (junction (at 55.88 57.15) (diameter 0) (color 0 0 0 0)
-  )
   (junction (at 236.22 44.45) (diameter 0) (color 0 0 0 0)
   )
@@
   (junction (at 182.88 110.49) (diameter 0) (color 0 0 0 0)
   )
+  (junction (at 59.69 46.99) (diameter 0) (color 0 0 0 0)
+  )
   (junction (at 227.33 35.56) (diameter 0) (color 0 0 0 0)
   )
@@
     (stroke (width 0) (type default))
   )
-  (wire (pts (xy 58.42 44.45) (xy 60.96 44.45))
+  (wire (pts (xy 59.69 44.45) (xy 60.96 44.45))
     (stroke (width 0) (type default))
   )
@@
     (stroke (width 0) (type default))
   )
+  (wire (pts (xy 59.69 49.53) (xy 59.69 46.99))
+    (stroke (width 0) (type default))
+  )
   (wire (pts (xy 259.08 144.78) (xy 259.08 143.51))
     (stroke (width 0) (type default))
@@
     (stroke (width 0) (type default))
   )
-  (wire (pts (xy 62.23 49.53) (xy 62.23 57.15))
-    (stroke (width 0) (type default))
-  )
   (wire (pts (xy 125.73 33.02) (xy 125.73 34.29))
     (stroke (width 0) (type default))
@@
     (stroke (width 0) (type default))
   )
-  (wire (pts (xy 55.88 46.99) (xy 58.42 46.99))
+  (wire (pts (xy 55.88 46.99) (xy 59.69 46.99))
     (stroke (width 0) (type default))
   )
@@
     (stroke (width 0) (type default))
   )
-  (wire (pts (xy 55.88 57.15) (xy 62.23 57.15))
-    (stroke (width 0) (type default))
-  )
   (wire (pts (xy 104.14 86.36) (xy 104.14 87.63))
     (stroke (width 0) (type default))
@@
     (stroke (width 0) (type default))
   )
-  (wire (pts (xy 58.42 46.99) (xy 58.42 44.45))
+  (wire (pts (xy 59.69 46.99) (xy 59.69 44.45))
     (stroke (width 0) (type default))
   )
@@
     (stroke (width 0) (type default))
   )
-  (wire (pts (xy 69.85 49.53) (xy 62.23 49.53))
+  (wire (pts (xy 59.69 49.53) (xy 69.85 49.53))
     (stroke (width 0) (type default))
   )
@@
     )
   )
-  (symbol (lib_id "Amplifier_Operational:OPA1692xD") (at 95.25 76.2 0) (unit 2)
+  (symbol (lib_id "Amplifier_Operational:OPA1692xD") (at 95.25 76.2 0) (unit 1)
     (in_bom yes) (on_board yes) (dnp no)
     (property "Reference" "U3" (at 93.98 69.215 0)
@@
       (project "tight-distortion"
         (path "/8747734a-25e9-406c-b9a5-cb27aff1316c/00000000-0000-0000-0000-0000667ed907"
-          (reference "U3") (unit 2)
+          (reference "U3") (unit 1)
         )
       )
@@
     )
   )
-  (symbol (lib_id "Amplifier_Operational:OPA1692xD") (at 200.66 86.36 0) (mirror x) (unit 1)
+  (symbol (lib_id "Amplifier_Operational:OPA1692xD") (at 200.66 86.36 0) (mirror x) (unit 2)
     (in_bom yes) (on_board yes) (dnp no)
     (property "Reference" "U3" (at 201.295 81.915 0)
@@
       (project "tight-distortion"
         (path "/8747734a-25e9-406c-b9a5-cb27aff1316c/00000000-0000-0000-0000-0000667ed907"
-          (reference "U3") (unit 1)
+          (reference "U3") (unit 2)
         )
       )
