File: tight-distortion.kicad_pcb (KiCad board)
At the start: 2 copper layers, 60 x 80 mm, 4 parts, among them J1 Barrel_Jack_Switch, J2 AudioJack_TRS, J3 AudioJack_TRS

Commit message: first PCB layout draft
Parts:
- added C1: 220pF, bca-footprints:C_Ceramic_L4.0mm_W2.5mm_P2.50mm, F.Cu at (12.4, -5.70)
- added C10: 100pF, bca-footprints:C_Ceramic_L4.0mm_W2.5mm_P2.50mm, F.Cu at (20.0, 8.30)
- added C11: 2.2nF, bca-footprints:C_Film_L7.2mm_W2.5mm_P5.00mm, F.Cu at (-4.00, -5.70)
- added C12: 10uF, bca-footprints:CP_Radial_D4.0mm_P1.50mm, F.Cu at (-6.30, 6.50)
- added C13: 100pF, bca-footprints:C_Ceramic_L4.0mm_W2.5mm_P2.50mm, F.Cu at (-3.90, -2.30)
- added C14: 4.7nF, bca-footprints:C_Film_L7.2mm_W2.5mm_P5.00mm, F.Cu at (-3.90, 10.4)
- added C15: 10uF, bca-footprints:CP_Radial_D4.0mm_P1.50mm, F.Cu at (-1.80, 6.50)
- added C16: 100pF, bca-footprints:C_Ceramic_L4.0mm_W2.5mm_P2.50mm, F.Cu at (-12.0, 17.9)
- added C17: 0.1uF, bca-footprints:C_Film_L7.2mm_W2.5mm_P5.00mm, F.Cu at (-20.4, -5.70)
- added C18: 0.1uF, bca-footprints:C_Film_L7.2mm_W2.5mm_P5.00mm, F.Cu at (-20.4, -2.30)
- added C19: 100pF, bca-footprints:C_Ceramic_L4.0mm_W2.5mm_P2.50mm, F.Cu at (-20.5, 5.50)
- added C2: 10nF, bca-footprints:C_Film_L7.2mm_W2.5mm_P5.00mm, F.Cu at (44.4, -3.40)
- added C20: 10nF, bca-footprints:C_Film_L7.2mm_W2.5mm_P5.00mm, F.Cu at (9.40, -14.2)
- added C21: 10nF, bca-footprints:C_Film_L7.2mm_W2.5mm_P5.00mm, F.Cu at (9.40, -17.4)
- added C22: 10nF, bca-footprints:C_Film_L7.2mm_W2.5mm_P5.00mm, F.Cu at (-10.0, -14.2)
- added C23: 10nF, bca-footprints:C_Film_L7.2mm_W2.5mm_P5.00mm, F.Cu at (-10.1, -17.4)
- added C24: 10nF, bca-footprints:C_Film_L7.2mm_W2.5mm_P5.00mm, F.Cu at (-20.1, -14.2)
- added C25: 10nF, bca-footprints:C_Film_L7.2mm_W2.5mm_P5.00mm, F.Cu at (-20.1, -17.4)
- added C26: 100pF, bca-footprints:C_Ceramic_L4.0mm_W2.5mm_P2.50mm, F.Cu at (-28.3, 3.90)
- added C27: 10nF, bca-footprints:C_Film_L7.2mm_W2.5mm_P5.00mm, F.Cu at (-20.5, 8.80)
- added C28: 100pF, bca-footprints:C_Ceramic_L4.0mm_W2.5mm_P2.50mm, F.Cu at (-20.4, 11.9)
- added C29: 0.1uF, bca-footprints:C_Film_L7.2mm_W2.5mm_P5.00mm, F.Cu at (-40.6, 4.80)
- added C3: 1nF, bca-footprints:C_Film_L7.2mm_W2.5mm_P5.00mm, F.Cu at (12.4, -2.30)
- added C30: 0.1uF, bca-footprints:C_Film_L7.2mm_W2.5mm_P5.00mm, F.Cu at (-40.6, 8.10)
- added C31: 0.1uF, bca-footprints:C_Film_L7.2mm_W2.5mm_P5.00mm, F.Cu at (-40.6, 19.5)
- added C32: 270pF, bca-footprints:C_Ceramic_L4.0mm_W2.5mm_P2.50mm, F.Cu at (-38.1, 12.2)
- added C33: 270pF, bca-footprints:C_Ceramic_L4.0mm_W2.5mm_P2.50mm, F.Cu at (-43.0, 12.2)
- added C34: 3.3nF, bca-footprints:C_Film_L7.2mm_W2.5mm_P5.00mm, F.Cu at (-40.6, 16.2)
- added C35: 100pF, bca-footprints:C_Ceramic_L4.0mm_W2.5mm_P2.50mm, F.Cu at (-49.6, -5.90)
- added C36: 0.1uF, bca-footprints:C_Film_L7.2mm_W2.5mm_P5.00mm, F.Cu at (-40.6, -12.9)
- added C37: 470uF, Capacitor_THT:CP_Radial_D8.0mm_P3.50mm, F.Cu at (-19.9, -38.0)
- added C38: 100uF, bca-footprints:CP_Radial_D6.3mm_P2.50mm, F.Cu at (16.0, -38.4)
- added C39: 10uF, bca-footprints:CP_Radial_D4.0mm_P1.50mm, F.Cu at (16.0, -32.0)
- added C4: 22nF, bca-footprints:C_Film_L7.2mm_W2.5mm_P5.00mm, F.Cu at (26.0, -3.40)
- added C40: 100uF, bca-footprints:CP_Radial_D6.3mm_P2.50mm, F.Cu at (-35.5, 35.5)
- added C41: 100nF, Capacitor_SMD:C_0805_2012Metric_Pad1.18x1.45mm_HandSolder, F.Cu at (-39.3, -6.00)
- added C42: 100nF, Capacitor_SMD:C_0805_2012Metric_Pad1.18x1.45mm_HandSolder, F.Cu at (-42.1, 1.60)
- added C43: 100nF, Capacitor_SMD:C_0805_2012Metric_Pad1.18x1.45mm_HandSolder, F.Cu at (1.40, -24.0)
- added C44: 100nF, Capacitor_SMD:C_0805_2012Metric_Pad1.18x1.45mm_HandSolder, F.Cu at (-1.40, -16.4)
- added C45: 100nF, Capacitor_SMD:C_0805_2012Metric_Pad1.18x1.45mm_HandSolder, F.Cu at (-17.0, -25.0)
- added C46: 100nF, Capacitor_SMD:C_0805_2012Metric_Pad1.18x1.45mm_HandSolder, F.Cu at (-22.9, -22.0)
- added C47: 100nF, Capacitor_SMD:C_0805_2012Metric_Pad1.18x1.45mm_HandSolder, F.Cu at (20.2, -32.0)
- added C48: 100nF, Capacitor_SMD:C_0805_2012Metric_Pad1.18x1.45mm_HandSolder, F.Cu at (26.5, -32.9)
- added C5: 2.2nF, bca-footprints:C_Film_L7.2mm_W2.5mm_P5.00mm, F.Cu at (12.4, 6.00)
- added C6: 10uF, bca-footprints:CP_Radial_D4.0mm_P1.50mm, F.Cu at (44.4, 4.10)
- added C7: 470pF, bca-footprints:C_Ceramic_L4.0mm_W2.5mm_P2.50mm, F.Cu at (12.4, 9.10)
- added C8: 2.2nF, bca-footprints:C_Film_L7.2mm_W2.5mm_P5.00mm, F.Cu at (26.0, 4.60)
- added C9: 10uF, bca-footprints:CP_Radial_D4.0mm_P1.50mm, F.Cu at (20.0, 12.1)
- added D1: 1N5819, Diode_SMD:D_SOD-123, F.Cu at (-8.80, -39.3)
- added D2: 1N5819, Diode_SMD:D_SOD-123, F.Cu at (-8.80, -36.7)
- added D3: 1N5819, Diode_SMD:D_SOD-123, F.Cu at (-14.1, -39.3)
- added D4: 1N5819, Diode_SMD:D_SOD-123, F.Cu at (-14.1, -36.7)
- added D5: LED, bca-footprints:LED_D5.0mm, B.Cu at (-45.0, 30.0)
- added J4: power-module, bca-footprints:Power-module, F.Cu at (0.00, 30.5)
- added J5: Conn_01x08, bca-footprints:Pin_Header_Straight_1x08_Pitch2.54mm, F.Cu at (40.0, 17.5)
- added Q1: MMBFJ202, Package_TO_SOT_SMD:SOT-23_Handsoldering, F.Cu at (12.5, 2.00)
- added Q10: BC848C, Package_TO_SOT_SMD:SOT-23_Handsoldering, F.Cu at (9.60, 29.9)
- added Q11: BC848C, Package_TO_SOT_SMD:SOT-23_Handsoldering, F.Cu at (3.80, 29.9)
- added Q12: BC848C, Package_TO_SOT_SMD:SOT-23_Handsoldering, F.Cu at (-2.00, 29.9)
- added Q13: BC848C, Package_TO_SOT_SMD:SOT-23_Handsoldering, F.Cu at (-7.80, 29.9)
- added Q2: MMBFJ202, Package_TO_SOT_SMD:SOT-23_Handsoldering, F.Cu at (12.4, 12.9)
- added Q3: MMBFJ202, Package_TO_SOT_SMD:SOT-23_Handsoldering, F.Cu at (-3.90, 2.00)
- added Q4: MMBFJ202, Package_TO_SOT_SMD:SOT-23_Handsoldering, F.Cu at (-3.90, 14.2)
- added Q5: BC848C, Package_TO_SOT_SMD:SOT-23_Handsoldering, F.Cu at (-20.4, 2.00)
- added Q6: LS844, Package_TO_SOT_SMD:SOT-23-6_Handsoldering, F.Cu at (-20.4, 15.4)
- added Q7: BC848C, Package_TO_SOT_SMD:SOT-23_Handsoldering, F.Cu at (-13.6, 29.9)
- added Q8: BC848C, Package_TO_SOT_SMD:SOT-23_Handsoldering, F.Cu at (-13.6, 26.0)
- added Q9: BC848C, Package_TO_SOT_SMD:SOT-23_Handsoldering, F.Cu at (15.4, 29.9)
- added R1: 68k, bca-footprints:R_L3.6mm_D1.6mm_P5.00mm_Horizontal, F.Cu at (4.50, -5.70)
- added R10: 15k, bca-footprints:R_L3.6mm_D1.6mm_P5.00mm_Horizontal, F.Cu at (4.50, 15.4)
- added R11: 2k, bca-footprints:R_L3.6mm_D1.6mm_P5.00mm_Horizontal, F.Cu at (4.50, 13.1)
- added R12: 220k, bca-footprints:R_L3.6mm_D1.6mm_P5.00mm_Horizontal, F.Cu at (-12.1, -5.70)
- added R13: 470k, bca-footprints:R_L3.6mm_D1.6mm_P5.00mm_Horizontal, F.Cu at (-12.1, -3.20)
- added R14: 47k, bca-footprints:R_L3.6mm_D1.6mm_P5.00mm_Horizontal, F.Cu at (50.5, -19.9)
- added R15: 47k, bca-footprints:R_L3.6mm_D1.6mm_P5.00mm_Horizontal, F.Cu at (-12.1, -0.80)
- added R16: 15k, bca-footprints:R_L3.6mm_D1.6mm_P5.00mm_Horizontal, F.Cu at (-12.1, 3.90)
- added R17: 2k, bca-footprints:R_L3.6mm_D1.6mm_P5.00mm_Horizontal, F.Cu at (-12.1, 1.50)
- added R18: 470k, bca-footprints:R_L3.6mm_D1.6mm_P5.00mm_Horizontal, F.Cu at (-12.1, 6.20)
- added R19: 220k, bca-footprints:R_L3.6mm_D1.6mm_P5.00mm_Horizontal, F.Cu at (-12.1, 8.50)
- added R2: 1M, bca-footprints:R_L3.6mm_D1.6mm_P5.00mm_Horizontal, F.Cu at (4.50, -3.20)
- added R20: 47k, bca-footprints:R_L3.6mm_D1.6mm_P5.00mm_Horizontal, F.Cu at (-12.1, 10.8)
- added R21: 7.5k, bca-footprints:R_L3.6mm_D1.6mm_P5.00mm_Horizontal, F.Cu at (-12.1, 15.4)
- added R22: 1k, bca-footprints:R_L3.6mm_D1.6mm_P5.00mm_Horizontal, F.Cu at (-12.1, 13.1)
- added R23: 470k, bca-footprints:R_L3.6mm_D1.6mm_P5.00mm_Horizontal, F.Cu at (-28.3, -5.70)
- added R24: 100k, bca-footprints:R_L3.6mm_D1.6mm_P5.00mm_Horizontal, F.Cu at (-28.3, -3.20)
- added R25: 15k, bca-footprints:R_L3.6mm_D1.6mm_P5.00mm_Horizontal, F.Cu at (-28.3, -0.80)
- added R26: 2k, bca-footprints:R_L3.6mm_D1.6mm_P5.00mm_Horizontal, F.Cu at (9.50, -20.5)
- added R27: 10k, bca-footprints:R_L3.6mm_D1.6mm_P5.00mm_Horizontal, F.Cu at (-28.2, 6.20)
- added R28: 2k, bca-footprints:R_L3.6mm_D1.6mm_P5.00mm_Horizontal, F.Cu at (9.50, -22.9)
- added R29: 2k, bca-footprints:R_L3.6mm_D1.6mm_P5.00mm_Horizontal, F.Cu at (-10.1, -20.5)
- added R3: 1M, bca-footprints:R_L3.6mm_D1.6mm_P5.00mm_Horizontal, F.Cu at (4.50, -0.80)
- added R30: 2k, bca-footprints:R_L3.6mm_D1.6mm_P5.00mm_Horizontal, F.Cu at (-10.1, -22.9)
- added R31: 2k, bca-footprints:R_L3.6mm_D1.6mm_P5.00mm_Horizontal, F.Cu at (-10.1, -25.3)
- added R32: 2k, bca-footprints:R_L3.6mm_D1.6mm_P5.00mm_Horizontal, F.Cu at (-10.1, -27.6)
- added R33: 10k, bca-footprints:R_L3.6mm_D1.6mm_P5.00mm_Horizontal, F.Cu at (-28.3, 1.50)
- added R34: 1M, bca-footprints:R_L3.6mm_D1.6mm_P5.00mm_Horizontal, F.Cu at (-28.2, 13.1)
- added R35: 10k, bca-footprints:R_L3.6mm_D1.6mm_P5.00mm_Horizontal, F.Cu at (-28.2, 15.4)
- added R36: 15k, bca-footprints:R_L3.6mm_D1.6mm_P5.00mm_Horizontal, F.Cu at (-28.2, 8.50)
- added R37: 15k, bca-footprints:R_L3.6mm_D1.6mm_P5.00mm_Horizontal, F.Cu at (-28.2, 10.7)
- added R38: 1M, bca-footprints:R_L3.6mm_D1.6mm_P5.00mm_Horizontal, F.Cu at (-28.2, 17.6)
- added R39: 100k, bca-footprints:R_L3.6mm_D1.6mm_P5.00mm_Horizontal, F.Cu at (-49.6, 3.90)
- added R4: 15k, bca-footprints:R_L3.6mm_D1.6mm_P5.00mm_Horizontal, F.Cu at (4.50, 3.90)
- added R40: 100k, bca-footprints:R_L3.6mm_D1.6mm_P5.00mm_Horizontal, F.Cu at (-49.6, 6.20)
- added R41: 10k, bca-footprints:R_L3.6mm_D1.6mm_P5.00mm_Horizontal, F.Cu at (-49.6, 15.4)
- added R42: 470R, bca-footprints:R_L3.6mm_D1.6mm_P5.00mm_Horizontal, F.Cu at (-49.6, 13.1)
- added R43: 100k, bca-footprints:R_L3.6mm_D1.6mm_P5.00mm_Horizontal, F.Cu at (-49.6, 8.50)
- added R44: 10k, bca-footprints:R_L3.6mm_D1.6mm_P5.00mm_Horizontal, F.Cu at (-49.6, -0.80)
- added R45: 10k, bca-footprints:R_L3.6mm_D1.6mm_P5.00mm_Horizontal, F.Cu at (-49.6, 1.50)
- added R46: 100k, bca-footprints:R_L3.6mm_D1.6mm_P5.00mm_Horizontal, F.Cu at (-49.6, -3.30)
- added R47: 100k, bca-footprints:R_L3.6mm_D1.6mm_P5.00mm_Horizontal, F.Cu at (-49.6, 10.7)
- added R48: 27k, bca-footprints:R_L3.6mm_D1.6mm_P5.00mm_Horizontal, F.Cu at (-14.7, 35.6)
- added R49: 470R, bca-footprints:R_L3.6mm_D1.6mm_P5.00mm_Horizontal, F.Cu at (-12.2, 35.6)
- added R5: 2k, bca-footprints:R_L3.6mm_D1.6mm_P5.00mm_Horizontal, F.Cu at (4.50, 1.50)
- added R50: 470R, bca-footprints:R_L3.6mm_D1.6mm_P5.00mm_Horizontal, F.Cu at (16.9, 35.6)
- added R51: 470R, bca-footprints:R_L3.6mm_D1.6mm_P5.00mm_Horizontal, F.Cu at (11.1, 35.6)
- added R52: 470R, bca-footprints:R_L3.6mm_D1.6mm_P5.00mm_Horizontal, F.Cu at (5.30, 35.6)
- added R53: 470R, bca-footprints:R_L3.6mm_D1.6mm_P5.00mm_Horizontal, F.Cu at (-0.50, 35.6)
- added R54: 470R, bca-footprints:R_L3.6mm_D1.6mm_P5.00mm_Horizontal, F.Cu at (-6.30, 35.6)
- added R55: 1k, bca-footprints:R_L3.6mm_D1.6mm_P5.00mm_Horizontal, F.Cu at (20.9, -38.4)
- added R56: 2k, bca-footprints:R_L3.6mm_D1.6mm_P5.00mm_Horizontal, F.Cu at (23.4, -38.4)
- added R57: 12k, bca-footprints:R_L3.6mm_D1.6mm_P5.00mm_Horizontal, F.Cu at (25.9, -38.4)
- added R58: 12k, bca-footprints:R_L3.6mm_D1.6mm_P5.00mm_Horizontal, F.Cu at (-30.1, 35.6)
- added R59: 3.3k, bca-footprints:R_L3.6mm_D1.6mm_P5.00mm_Horizontal, F.Cu at (-27.3, 35.6)
- added R6: 220k, bca-footprints:R_L3.6mm_D1.6mm_P5.00mm_Horizontal, F.Cu at (4.50, 6.20)
- added R60: 33k, bca-footprints:R_L3.6mm_D1.6mm_P5.00mm_Horizontal, F.Cu at (48.8, 13.6)
- added R61: 470R, bca-footprints:R_L3.6mm_D1.6mm_P5.00mm_Horizontal, F.Cu at (-2.70, 35.6)
- added R62: 470R, bca-footprints:R_L3.6mm_D1.6mm_P5.00mm_Horizontal, F.Cu at (-8.60, 35.6)
- added R7: 220k, bca-footprints:R_L3.6mm_D1.6mm_P5.00mm_Horizontal, F.Cu at (4.50, 8.50)
- added R8: 47k, bca-footprints:R_L3.6mm_D1.6mm_P5.00mm_Horizontal, F.Cu at (52.8, -19.9)
- added R9: 47k, bca-footprints:R_L3.6mm_D1.6mm_P5.00mm_Horizontal, F.Cu at (4.50, 10.8)
- added RV1: 500kA, bca-footprints:R_POT_DUAL, F.Cu at (45.0, -26.0)
- added RV2: 100kB, bca-footprints:R_POT, F.Cu at (22.5, -26.0)
- added RV3: 100kB, bca-footprints:R_POT, F.Cu at (0.00, -26.0)
- added RV4: 100kB, bca-footprints:R_POT, F.Cu at (-22.5, -26.0)
- added RV5: 100kA, bca-footprints:R_POT, F.Cu at (-45.0, -26.0)
- added SW1: SW_DPDT_x2, bca-footprints:SW_Toggle_DPDT_SolderLug, F.Cu at (35.0, 0.00)
- added SW2: SW_SPDT, bca-footprints:SW_Toggle_SPDT_SolderLug, F.Cu at (50.0, 0.00)
- added SW3: SW_SPDT, bca-footprints:SW_Toggle_SPDT_SolderLug, F.Cu at (20.0, 0.00)
- added U1: TLV9302, Package_SO:SOIC-8_3.9x4.9mm_P1.27mm, F.Cu at (0.00, -20.1)
- added U2: TLV9301, Package_TO_SOT_SMD:SOT-23-5, F.Cu at (-20.0, -23.0)
- added U3: OPA1692xD, Package_SO:SOIC-8_3.9x4.9mm_P1.27mm, F.Cu at (-40.7, -2.20)
- added U4: TLV9301, Package_TO_SOT_SMD:SOT-23-5, F.Cu at (23.4, -31.9)
- moved G1 28.2 mm to (53.4, -30.0)
- moved J2 27.4 mm to (-38.0, -30.0)
- moved J3 27.4 mm to (38.0, -30.0)
- moved J1 14.2 mm to (0.00, -43.5)
Connections:
- J1 pad 1: Net-(J1-Pad1) -> Net-(D2-Pad1)
- J2 pad 2: Net-(J1-Pad1) -> Earth
- J2 pad 5: Net-(J2-Pad5) -> Earth
Routing:
- net Earth: track 0.00 -> 84.5 mm
- net Net-(C37-Pad1): track 0.00 -> 82.0 mm
- net -15V: track 0.00 -> 2.54 mm
- net +15V: track 0.00 -> 2.54 mm
- added copper zone on In1.Cu, net Earth
Other:
- board size 60 x 80 mm -> 110 x 84.3 mm
- copper layers 2 -> 4
- net class Default: trace_width 0.15 -> 0.25
- net class PWR removed
- rule trace_min: 0.15 -> 0.2
- rule via_min_drill: 0.4 -> 0.3
- rule via_min_size: 0.8 -> 0.4
- board text added: "JLCJLCJLCJLC"
- board text added: "LTP CS"
- board text added: "Q4 CS"

Commit message: first pass of routing PCB
Parts:
- moved C12 4.50 mm to (-1.80, 6.50)
- moved C15 4.50 mm to (-6.30, 6.50)
- moved C38 1.84 mm to (14.2, -38.0)
- moved C39 1.84 mm to (14.2, -31.6)
- moved C47 1.84 mm to (18.4, -31.6)
- moved C48 1.84 mm to (24.7, -32.5)
- moved R55 1.84 mm to (19.1, -38.0)
- moved R56 1.84 mm to (21.6, -38.0)
- moved R57 1.84 mm to (24.1, -38.0)
- moved U4 1.84 mm to (21.6, -31.5)
- turned C18 to 180 degrees
- turned C19 to 0 degrees
- turned C2 to 90 degrees
- turned R15 to 0 degrees
- turned R27 to 0 degrees
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Routing:
- net /input_jack: track 0.00 -> 190.2 mm
- net /return: track 0.00 -> 168.2 mm
- net /Signal Path/-VREF0: track 0.00 -> 140.6 mm, vias 0 -> 2
- net /LED+: track 0.00 -> 120.5 mm
- net Net-(C19-Pad2): track 0.00 -> 99.1 mm
- net /Signal Path/ccs0: track 0.00 -> 89.6 mm, vias 0 -> 2
- net /output_jack: track 0.00 -> 77.5 mm
- net Net-(C26-Pad1): track 0.00 -> 71.2 mm
- net Net-(C7-Pad2): track 0.00 -> 70.5 mm
- net Net-(R15-Pad1): track 0.00 -> 67.2 mm
- net Net-(C8-Pad1): track 0.00 -> 63.3 mm
- net Net-(R12-Pad2): track 0.00 -> 60.3 mm
- net Net-(Q1-Pad2): track 0.00 -> 59.1 mm, vias 0 -> 1
- net /send: track 0.00 -> 56.7 mm, vias 0 -> 1
- net Net-(C2-Pad1): track 0.00 -> 56.0 mm
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- added copper zone on In2.Cu, net +15V
- added copper zone on In2.Cu, net -15V
- added copper zone on F.Cu, net /Signal Path/-VREF1
- added copper zone on F.Cu, net Earth
- added copper zone on F.Cu, net Net-(C37-Pad1)
- added copper zone on F.Cu, net Net-(C38-Pad2)
- added copper zone on F.Cu, net Net-(D1-Pad1)
- added copper zone on F.Cu, net Net-(D2-Pad1)
Other:
- board text added: "BCA Distortion v1.0.0; Dec 2023"
- board text added: "Designed & Assembled in St. John's, NL"
- board text added: "LTP"
- board text added: "Q1"
- board text added: "Q2"
- board text added: "Q3"
- board text added: "Q4"
- board text removed: "LTP CS"
- board text removed: "Q4 CS"

Commit message: corrected & finalized PCB
Parts:
- added C49: 1uF, Capacitor_SMD:C_0805_2012Metric_Pad1.18x1.45mm_HandSolder, F.Cu at (-26.0, -32.6)
Connections:
- Q10 pad 1: /Signal Path/ccs1 -> Net-(Q10-Pad1)
- Q10 pad 3: Net-(Q10-Pad3) -> /Signal Path/ccs1
- Q11 pad 1: /Signal Path/ccs2 -> Net-(Q10-Pad1)
- Q11 pad 2: Net-(Q10-Pad2) -> Net-(Q11-Pad2)
- Q11 pad 3: Net-(Q11-Pad3) -> /Signal Path/ccs2
- Q12 pad 1: /Signal Path/ccs3 -> Net-(Q10-Pad1)
- Q12 pad 2: Net-(Q10-Pad2) -> Net-(Q12-Pad2)
- Q12 pad 3: Net-(Q12-Pad3) -> /Signal Path/ccs3
- Q13 pad 1: /Signal Path/ccs4 -> Net-(Q10-Pad1)
- Q13 pad 2: Net-(Q10-Pad2) -> Net-(Q13-Pad2)
- Q13 pad 3: Net-(Q13-Pad3) -> /Signal Path/ccs4
- Q7 pad 1: Net-(Q7-Pad1) -> Net-(Q10-Pad1)
- Q7 pad 2: Net-(Q10-Pad2) -> Net-(Q7-Pad2)
- Q8 pad 1: Earth -> Net-(Q7-Pad3)
- Q8 pad 2: Net-(Q7-Pad1) -> Net-(Q10-Pad1)
- Q8 pad 3: Net-(Q10-Pad2) -> Earth
- Q9 pad 1: /Signal Path/ccs0 -> Net-(Q10-Pad1)
- Q9 pad 2: Net-(Q10-Pad2) -> Net-(Q9-Pad2)
- Q9 pad 3: Net-(Q9-Pad3) -> /Signal Path/ccs0
- R48 pad 2: Net-(Q7-Pad1) -> Net-(Q7-Pad3)
- R49 pad 1: Net-(Q7-Pad3) -> Net-(Q7-Pad2)
- R50 pad 1: Net-(Q9-Pad3) -> Net-(Q9-Pad2)
- R51 pad 1: Net-(Q10-Pad3) -> Net-(Q10-Pad2)
- R52 pad 1: Net-(Q11-Pad3) -> Net-(Q11-Pad2)
- R53 pad 1: Net-(Q12-Pad3) -> Net-(Q12-Pad2)
- R54 pad 1: Net-(Q13-Pad3) -> Net-(Q13-Pad2)
- R61 pad 1: Net-(Q12-Pad3) -> Net-(Q12-Pad2)
- R62 pad 1: Net-(Q13-Pad3) -> Net-(Q13-Pad2)
Routing:
- net Net-(Q10-Pad2): track 54.7 -> 4.34 mm
- net Net-(Q10-Pad1): track 0.00 -> 37.7 mm, vias 0 -> 5
- net Net-(Q7-Pad3): track 3.24 -> 16.1 mm
- net Net-(Q7-Pad1): track 9.65 -> 0.00 mm
- net Net-(Q13-Pad3): track 5.50 -> 0.00 mm
- net Net-(Q12-Pad3): track 5.40 -> 0.00 mm
- net /Signal Path/ccs0: track 89.6 -> 94.9 mm
- net Net-(Q13-Pad2): track 0.00 -> 4.84 mm
- net Net-(Q12-Pad2): track 0.00 -> 4.78 mm
- net Net-(Q9-Pad2): track 0.00 -> 4.58 mm
- net Net-(Q7-Pad2): track 0.00 -> 4.48 mm
- net /Signal Path/ccs1: track 18.4 -> 22.8 mm
- net Net-(Q11-Pad2): track 0.00 -> 4.40 mm
- net /Signal Path/ccs3: track 36.4 -> 40.6 mm
- net Net-(Q9-Pad3): track 3.20 -> 0.00 mm
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
Commit message: gerbers
Other:
- board text added: "ALL 100kB POTS USE CENTER DETENT"
- board text added: "ALL SWITCHES ON-ON"
Changed lines of the file:
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@@
   (general
     (thickness 1.6)
-    (drawings 60)
+    (drawings 62)
     (tracks 770)
     (zones 0)
@@
       (effects (font (size 0.5 0.5) (thickness 0.08)))
     )
-    (pad 1 smd roundrect (at -1.0375 0 180) (size 1.175 1.45) (layers F.Cu F.Paste F.Mask) (roundrect_rratio 0.212766)
+    (pad 1 smd roundrect (at -1.0375 0 180) (size 1.175 1.45) (layers F.Cu F.Paste F.Mask) (roundrect_rratio 0.2127659574468085)
       (net 14 +15V))
-    (pad 2 smd roundrect (at 1.0375 0 180) (size 1.175 1.45) (layers F.Cu F.Paste F.Mask) (roundrect_rratio 0.212766)
+    (pad 2 smd roundrect (at 1.0375 0 180) (size 1.175 1.45) (layers F.Cu F.Paste F.Mask) (roundrect_rratio 0.2127659574468085)
       (net 1 Earth))
     (model ${KISYS3DMOD}/Capacitor_SMD.3dshapes/C_0805_2012Metric.wrl
@@
       (effects (font (size 0.5 0.5) (thickness 0.08)))
     )
-    (pad 2 smd roundrect (at 1.0375 0 180) (size 1.175 1.45) (layers F.Cu F.Paste F.Mask) (roundrect_rratio 0.212766)
+    (pad 2 smd roundrect (at 1.0375 0 180) (size 1.175 1.45) (layers F.Cu F.Paste F.Mask) (roundrect_rratio 0.2127659574468085)
       (net 15 -15V))
-    (pad 1 smd roundrect (at -1.0375 0 180) (size 1.175 1.45) (layers F.Cu F.Paste F.Mask) (roundrect_rratio 0.212766)
+    (pad 1 smd roundrect (at -1.0375 0 180) (size 1.175 1.45) (layers F.Cu F.Paste F.Mask) (roundrect_rratio 0.2127659574468085)
       (net 1 Earth))
     (model ${KISYS3DMOD}/Capacitor_SMD.3dshapes/C_0805_2012Metric.wrl
@@
       (effects (font (size 0.5 0.5) (thickness 0.08)))
     )
-    (pad 1 smd roundrect (at -1.0375 0 180) (size 1.175 1.45) (layers F.Cu F.Paste F.Mask) (roundrect_rratio 0.212766)
+    (pad 1 smd roundrect (at -1.0375 0 180) (size 1.175 1.45) (layers F.Cu F.Paste F.Mask) (roundrect_rratio 0.2127659574468085)
       (net 14 +15V))
-    (pad 2 smd roundrect (at 1.0375 0 180) (size 1.175 1.45) (layers F.Cu F.Paste F.Mask) (roundrect_rratio 0.212766)
+    (pad 2 smd roundrect (at 1.0375 0 180) (size 1.175 1.45) (layers F.Cu F.Paste F.Mask) (roundrect_rratio 0.2127659574468085)
       (net 1 Earth))
     (model ${KISYS3DMOD}/Capacitor_SMD.3dshapes/C_0805_2012Metric.wrl
@@
       (effects (font (size 0.5 0.5) (thickness 0.08)))
     )
-    (pad 2 smd roundrect (at 1.0375 0 180) (size 1.175 1.45) (layers F.Cu F.Paste F.Mask) (roundrect_rratio 0.212766)
+    (pad 2 smd roundrect (at 1.0375 0 180) (size 1.175 1.45) (layers F.Cu F.Paste F.Mask) (roundrect_rratio 0.2127659574468085)
       (net 15 -15V))
-    (pad 1 smd roundrect (at -1.0375 0 180) (size 1.175 1.45) (layers F.Cu F.Paste F.Mask) (roundrect_rratio 0.212766)
+    (pad 1 smd roundrect (at -1.0375 0 180) (size 1.175 1.45) (layers F.Cu F.Paste F.Mask) (roundrect_rratio 0.2127659574468085)
       (net 1 Earth))
     (model ${KISYS3DMOD}/Capacitor_SMD.3dshapes/C_0805_2012Metric.wrl
@@
       (effects (font (size 0.5 0.5) (thickness 0.08)))
     )
-    (pad 1 smd roundrect (at -1.0375 0 90) (size 1.175 1.45) (layers F.Cu F.Paste F.Mask) (roundrect_rratio 0.212766)
+    (pad 1 smd roundrect (at -1.0375 0 90) (size 1.175 1.45) (layers F.Cu F.Paste F.Mask) (roundrect_rratio 0.2127659574468085)
       (net 14 +15V))
-    (pad 2 smd roundrect (at 1.0375 0 90) (size 1.175 1.45) (layers F.Cu F.Paste F.Mask) (roundrect_rratio 0.212766)
+    (pad 2 smd roundrect (at 1.0375 0 90) (size 1.175 1.45) (layers F.Cu F.Paste F.Mask) (roundrect_rratio 0.2127659574468085)
       (net 1 Earth))
     (model ${KISYS3DMOD}/Capacitor_SMD.3dshapes/C_0805_2012Metric.wrl
@@
       (effects (font (size 0.5 0.5) (thickness 0.08)))
     )
-    (pad 2 smd roundrect (at 1.0375 0 90) (size 1.175 1.45) (layers F.Cu F.Paste F.Mask) (roundrect_rratio 0.212766)
+    (pad 2 smd roundrect (at 1.0375 0 90) (size 1.175 1.45) (layers F.Cu F.Paste F.Mask) (roundrect_rratio 0.2127659574468085)
       (net 15 -15V))
-    (pad 1 smd roundrect (at -1.0375 0 90) (size 1.175 1.45) (layers F.Cu F.Paste F.Mask) (roundrect_rratio 0.212766)
+    (pad 1 smd roundrect (at -1.0375 0 90) (size 1.175 1.45) (layers F.Cu F.Paste F.Mask) (roundrect_rratio 0.2127659574468085)
       (net 1 Earth))
     (model ${KISYS3DMOD}/Capacitor_SMD.3dshapes/C_0805_2012Metric.wrl
@@
       (effects (font (size 0.5 0.5) (thickness 0.08)))
     )
-    (pad 1 smd roundrect (at -1.0375 0 90) (size 1.175 1.45) (layers F.Cu F.Paste F.Mask) (roundrect_rratio 0.212766)
+    (pad 1 smd roundrect (at -1.0375 0 90) (size 1.175 1.45) (layers F.Cu F.Paste F.Mask) (roundrect_rratio 0.2127659574468085)
       (net 14 +15V))
-    (pad 2 smd roundrect (at 1.0375 0 90) (size 1.175 1.45) (layers F.Cu F.Paste F.Mask) (roundrect_rratio 0.212766)
+    (pad 2 smd roundrect (at 1.0375 0 90) (size 1.175 1.45) (layers F.Cu F.Paste F.Mask) (roundrect_rratio 0.2127659574468085)
       (net 1 Earth))
     (model ${KISYS3DMOD}/Capacitor_SMD.3dshapes/C_0805_2012Metric.wrl
@@
       (effects (font (size 0.5 0.5) (thickness 0.08)))
     )
-    (pad 2 smd roundrect (at 1.0375 0 270) (size 1.175 1.45) (layers F.Cu F.Paste F.Mask) (roundrect_rratio 0.212766)
+    (pad 2 smd roundrect (at 1.0375 0 270) (size 1.175 1.45) (layers F.Cu F.Paste F.Mask) (roundrect_rratio 0.2127659574468085)
       (net 15 -15V))
-    (pad 1 smd roundrect (at -1.0375 0 270) (size 1.175 1.45) (layers F.Cu F.Paste F.Mask) (roundrect_rratio 0.212766)
+    (pad 1 smd roundrect (at -1.0375 0 270) (size 1.175 1.45) (layers F.Cu F.Paste F.Mask) (roundrect_rratio 0.2127659574468085)
       (net 1 Earth))
     (model ${KISYS3DMOD}/Capacitor_SMD.3dshapes/C_0805_2012Metric.wrl
@@
       (effects (font (size 0.5 0.5) (thickness 0.08)))
     )
-    (pad 1 smd roundrect (at -1.0375 0 180) (size 1.175 1.45) (layers F.Cu F.Paste F.Mask) (roundrect_rratio 0.212766)
+    (pad 1 smd roundrect (at -1.0375 0 180) (size 1.175 1.45) (layers F.Cu F.Paste F.Mask) (roundrect_rratio 0.2127659574468085)
       (net 62 "Net-(C37-Pad1)"))
-    (pad 2 smd roundrect (at 1.0375 0 180) (size 1.175 1.45) (layers F.Cu F.Paste F.Mask) (roundrect_rratio 0.212766)
+    (pad 2 smd roundrect (at 1.0375 0 180) (size 1.175 1.45) (layers F.Cu F.Paste F.Mask) (roundrect_rratio 0.2127659574468085)
       (net 1 Earth))
     (model ${KISYS3DMOD}/Capacitor_SMD.3dshapes/C_0805_2012Metric.wrl
@@
     )
   )
+  (gr_text "ALL SWITCHES ON-ON" (at 34.9 9.3) (layer B.SilkS)
+    (effects (font (size 1 1) (thickness 0.15)) (justify mirror))
+  )
+  (gr_text "ALL 100kB POTS USE\nCENTER DETENT" (at 2.5 -39.9) (layer B.SilkS)
+    (effects (font (size 1 1) (thickness 0.15)) (justify mirror))
+  )
   (gr_text Q1 (at 16.9 40) (layer F.SilkS)
     (effects (font (size 1 1) (thickness 0.15)))
@@
     (effects (font (size 1 1) (thickness 0.15)) (justify left))
   )
-  (gr_text "BCA Distortion\nv1.0.0; Dec 2023" (at -51.8 -30 90) (layer F.SilkS)
+  (gr_text "BCA Distortion\nv1.0.0; Dec 2023" (at -51.4 -26.8 90) (layer F.SilkS)
     (effects (font (size 1 1) (thickness 0.15)))
   )

Commit message: development checkpoint
Parts:
- C20, C21: value 10nF -> 0.15uF
- C22: value 10nF -> 47nF
- C23, C24: value 10nF -> 22nF
- C25: value 10nF -> 15nF
- R26, R29, R31: value 2k -> 680R
- R27, R33: value 10k -> 2.7k
- R28, R30: value 2k -> 68k
- R32: value 2k -> 82k
- R54: value 470R -> 220R
- R62: value 470R -> 330R
- RV2, RV3, RV4: value 100kB -> 20kW
Changed lines of the file:
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@@
   )
   (setup
-    (last_trace_width 0.5)
+    (last_trace_width 0.25)
     (user_trace_width 0.5)
     (user_trace_width 1)
@@
       (effects (font (size 1 1) (thickness 0.15)))
     )
-    (fp_text value 10nF (at 0 2.56) (layer F.Fab) hide
+    (fp_text value 0.15uF (at 0 2.56) (layer F.Fab) hide
       (effects (font (size 1 1) (thickness 0.15)))
     )
@@
       (effects (font (size 1 1) (thickness 0.15)))
     )
-    (fp_text value 10nF (at 0 2.56) (layer F.Fab) hide
+    (fp_text value 0.15uF (at 0 2.56) (layer F.Fab) hide
       (effects (font (size 1 1) (thickness 0.15)))
     )
@@
       (effects (font (size 1 1) (thickness 0.15)))
     )
-    (fp_text value 10nF (at 0 2.56) (layer F.Fab) hide
+    (fp_text value 47nF (at 0 2.56) (layer F.Fab) hide
       (effects (font (size 1 1) (thickness 0.15)))
     )
@@
       (effects (font (size 1 1) (thickness 0.15)))
     )
-    (fp_text value 10nF (at 0 2.56) (layer F.Fab) hide
+    (fp_text value 22nF (at 0 2.56) (layer F.Fab) hide
       (effects (font (size 1 1) (thickness 0.15)))
     )
@@
       (effects (font (size 1 1) (thickness 0.15)))
     )
-    (fp_text value 10nF (at 0 2.56) (layer F.Fab) hide
+    (fp_text value 22nF (at 0 2.56) (layer F.Fab) hide
       (effects (font (size 1 1) (thickness 0.15)))
     )
@@
       (effects (font (size 1 1) (thickness 0.15)))
     )
-    (fp_text value 10nF (at 0 2.56) (layer F.Fab) hide
+    (fp_text value 15nF (at 0 2.56) (layer F.Fab) hide
       (effects (font (size 1 1) (thickness 0.15)))
     )
@@
       (effects (font (size 1 1) (thickness 0.15)))
     )
-    (fp_text value 2k (at 2.5 1.86) (layer F.Fab) hide
+    (fp_text value 680R (at 2.5 1.86) (layer F.Fab) hide
       (effects (font (size 1 1) (thickness 0.15)))
     )
@@
       (effects (font (size 1 1) (thickness 0.15)))
     )
-    (fp_text value 10k (at 2.5 1.86) (layer F.Fab) hide
+    (fp_text value 2.7k (at 2.5 1.86) (layer F.Fab) hide
       (effects (font (size 1 1) (thickness 0.15)))
     )
@@
       (effects (font (size 1 1) (thickness 0.15)))
     )
-    (fp_text value 2k (at 2.5 1.86) (layer F.Fab) hide
+    (fp_text value 68k (at 2.5 1.86) (layer F.Fab) hide
       (effects (font (size 1 1) (thickness 0.15)))
     )
@@
       (effects (font (size 1 1) (thickness 0.15)))
     )
-    (fp_text value 2k (at 2.5 1.86) (layer F.Fab) hide
+    (fp_text value 680R (at 2.5 1.86) (layer F.Fab) hide
       (effects (font (size 1 1) (thickness 0.15)))
     )
@@
       (effects (font (size 1 1) (thickness 0.15)))
     )
-    (fp_text value 2k (at 2.5 1.86) (layer F.Fab) hide
+    (fp_text value 68k (at 2.5 1.86) (layer F.Fab) hide
       (effects (font (size 1 1) (thickness 0.15)))
     )
@@
       (effects (font (size 1 1) (thickness 0.15)))
     )
-    (fp_text value 2k (at 2.5 1.86) (layer F.Fab) hide
+    (fp_text value 680R (at 2.5 1.86) (layer F.Fab) hide
       (effects (font (size 1 1) (thickness 0.15)))
     )
@@
       (effects (font (size 1 1) (thickness 0.15)))
     )
-    (fp_text value 2k (at 2.5 1.86) (layer F.Fab) hide
+    (fp_text value 82k (at 2.5 1.86) (layer F.Fab) hide
       (effects (font (size 1 1) (thickness 0.15)))
     )
@@
       (effects (font (size 1 1) (thickness 0.15)))
     )
-    (fp_text value 10k (at 2.5 1.86) (layer F.Fab) hide
+    (fp_text value 2.7k (at 2.5 1.86) (layer F.Fab) hide
       (effects (font (size 1 1) (thickness 0.15)))
     )
@@
       (effects (font (size 1 1) (thickness 0.15)))
     )
-    (fp_text value 470R (at 2.5 1.86 90) (layer F.Fab) hide
+    (fp_text value 220R (at 2.5 1.86 90) (layer F.Fab) hide
       (effects (font (size 1 1) (thickness 0.15)))
     )
@@
       (effects (font (size 1 1) (thickness 0.15)) (justify mirror))
     )
-    (fp_text value 100kB (at 0 5 180) (layer B.SilkS)
+    (fp_text value 20kW (at 0 5 180) (layer B.SilkS)
       (effects (font (size 1 1) (thickness 0.15)) (justify mirror))
     )
@@
       (effects (font (size 1 1) (thickness 0.15)) (justify mirror))
     )
-    (fp_text value 100kB (at 0 5 180) (layer B.SilkS)
+    (fp_text value 20kW (at 0 5 180) (layer B.SilkS)
       (effects (font (size 1 1) (thickness 0.15)) (justify mirror))
     )
@@
       (effects (font (size 1 1) (thickness 0.15)) (justify mirror))
     )
-    (fp_text value 100kB (at 0 5 180) (layer B.SilkS)
+    (fp_text value 20kW (at 0 5 180) (layer B.SilkS)
       (effects (font (size 1 1) (thickness 0.15)) (justify mirror))
     )
@@
       (effects (font (size 1 1) (thickness 0.15)))
     )
-    (fp_text value 470R (at 2.5 1.86 90) (layer F.Fab) hide
+    (fp_text value 330R (at 2.5 1.86 90) (layer F.Fab) hide
       (effects (font (size 1 1) (thickness 0.15)))
     )
