File: tight-distortion.kicad_pcb (KiCad board)
At the start: 4 copper layers, 110 x 84.3 mm, 147 parts, among them J1 Barrel_Jack_Switch, J2 AudioJack_TRS, J3 AudioJack_TRS, J4 power-module, J5 Conn_01x08, Q1 MMBFJ202, Q10 BC848C, Q11 BC848C, Q12 BC848C, Q13 BC848C, Q2 MMBFJ202, Q3 MMBFJ202, Q4 MMBFJ202, Q5 BC848C, Q6 LS844, Q7 BC848C, Q8 BC848C, Q9 BC848C, SW1 SW_DPDT_x2, SW2 SW_SPDT, SW3 SW_SPDT, U1 TLV9302, U2 TLV9301, U3 OPA1692xD, U4 TLV9301

Commit message: start of PCB re-route
Parts:
- removed C49: 1uF, Capacitor_SMD:C_0805_2012Metric_Pad1.18x1.45mm_HandSolder
- removed U2: TLV9301, Package_TO_SOT_SMD:SOT-23-5
- added D6: LED_Dual_AAK, bca-footprints:LED_D5.0mm-3, B.Cu at (-22.5, 17.5)
- added R63: 39k, bca-footprints:R_L3.6mm_D1.6mm_P5.00mm_Horizontal, F.Cu at (-50.0, 14.6)
- C1, C28, C7: footprint bca-footprints:C_Ceramic_L4.0mm_W2.5mm_P2.50mm -> Capacitor_SMD:C_0603_1608Metric_Pad1.08x0.95mm_HandSolder
- C10: value 100pF -> 820pF; footprint bca-footprints:C_Ceramic_L4.0mm_W2.5mm_P2.50mm -> Capacitor_SMD:C_0603_1608Metric_Pad1.08x0.95mm_HandSolder
- C11: value 2.2nF -> 4.7nF
- C12: value 10uF -> 470pF; footprint bca-footprints:CP_Radial_D4.0mm_P1.50mm -> Capacitor_SMD:C_0603_1608Metric_Pad1.08x0.95mm_HandSolder
- C13: value 100pF -> 10uF; footprint bca-footprints:C_Ceramic_L4.0mm_W2.5mm_P2.50mm -> bca-footprints:CP_Radial_D4.0mm_P1.50mm
- C14: value 4.7nF -> 820pF; footprint bca-footprints:C_Film_L7.2mm_W2.5mm_P5.00mm -> Capacitor_SMD:C_0603_1608Metric_Pad1.08x0.95mm_HandSolder
- C15: value 10uF -> 4.7nF; footprint bca-footprints:CP_Radial_D4.0mm_P1.50mm -> bca-footprints:C_Film_L7.2mm_W2.5mm_P5.00mm
- C16: value 100pF -> 470pF; footprint bca-footprints:C_Ceramic_L4.0mm_W2.5mm_P2.50mm -> Capacitor_SMD:C_0603_1608Metric_Pad1.08x0.95mm_HandSolder
- C17: value 0.1uF -> 10uF; footprint bca-footprints:C_Film_L7.2mm_W2.5mm_P5.00mm -> bca-footprints:CP_Radial_D4.0mm_P1.50mm
- C18: value 0.1uF -> 820pF; footprint bca-footprints:C_Film_L7.2mm_W2.5mm_P5.00mm -> Capacitor_SMD:C_0603_1608Metric_Pad1.08x0.95mm_HandSolder
- C19: value 100pF -> 0.1uF; footprint bca-footprints:C_Ceramic_L4.0mm_W2.5mm_P2.50mm -> bca-footprints:C_Film_L7.2mm_W2.5mm_P5.00mm
- C20: value 0.15uF -> 10nF
- C21: value 0.15uF -> 4.7nF
- C22: value 47nF -> 39nF
- C23, C24: value 22nF -> 56nF
- C25: value 15nF -> 39nF
- C26: value 100pF -> 4.7nF; footprint bca-footprints:C_Ceramic_L4.0mm_W2.5mm_P2.50mm -> bca-footprints:C_Film_L7.2mm_W2.5mm_P5.00mm
- C32, C33: value 270pF -> 68pF; footprint bca-footprints:C_Ceramic_L4.0mm_W2.5mm_P2.50mm -> Capacitor_SMD:C_0603_1608Metric_Pad1.08x0.95mm_HandSolder
- C34: value 3.3nF -> 0.15uF
- C35: value 100pF -> 1nF; footprint bca-footprints:C_Ceramic_L4.0mm_W2.5mm_P2.50mm -> bca-footprints:C_Film_L7.2mm_W2.5mm_P5.00mm
- C36: value 0.1uF -> 3.3nF
- C37: value 470uF -> 0.1uF; footprint Capacitor_THT:CP_Radial_D8.0mm_P3.50mm -> bca-footprints:C_Film_L7.2mm_W2.5mm_P5.00mm
- C41, C42, C43, C44, C45, C46: footprint Capacitor_SMD:C_0805_2012Metric_Pad1.18x1.45mm_HandSolder -> Capacitor_SMD:C_0603_1608Metric_Pad1.08x0.95mm_HandSolder
- C47: value 100nF -> 470uF; footprint Capacitor_SMD:C_0805_2012Metric_Pad1.18x1.45mm_HandSolder -> Capacitor_THT:CP_Radial_D8.0mm_P3.50mm
- C48: value 100nF -> 1uF
- C8: value 2.2nF -> 1nF
- J4: value power-module -> Conn_01x08; footprint bca-footprints:Power-module -> bca-footprints:Pin_Header_Straight_1x08_Pitch2.54mm
- J5: value Conn_01x08 -> power-module; footprint bca-footprints:Pin_Header_Straight_1x08_Pitch2.54mm -> bca-footprints:Power-module
- R12: value 220k -> 470k
- R13, R18: value 470k -> 220k
- R14, R8, R9: value 47k -> 220k
- R15: value 47k -> 15k
- R16: value 15k -> 2k
- R17: value 2k -> 470k
- R19: value 220k -> 7.5k
- R20: value 47k -> 1k
- R21: value 7.5k -> 470k
- R22: value 1k -> 220k
- R23: value 470k -> 15k
- R24: value 100k -> 3.9k
- R25, R36: value 15k -> 1M
- R26: value 680R -> 1k
- R27: value 2.7k -> 82k
- R28: value 68k -> 680R
- R29: value 680R -> 47k
- R30: value 68k -> 1k
- R31: value 680R -> 3.9k
- R32: value 82k -> 1M
- R33: value 2.7k -> 10k
- R34: value 1M -> 15k
- R35: value 10k -> 15k
- R37: value 15k -> 680k
- R38: value 1M -> 680k
- R39: value 100k -> 15k
- R40: value 100k -> 39k
- R41: value 10k -> 470R
- R42: value 470R -> 10k
- R43: value 100k -> 10k
- R44: value 10k -> 2.2k
- R45: value 10k -> 39k
- R47: value 100k -> 27k; footprint bca-footprints:R_L3.6mm_D1.6mm_P5.00mm_Horizontal -> Resistor_SMD:R_0603_1608Metric_Pad0.98x0.95mm_HandSolder
- R48: value 27k -> 470R; footprint bca-footprints:R_L3.6mm_D1.6mm_P5.00mm_Horizontal -> Resistor_SMD:R_0603_1608Metric_Pad0.98x0.95mm_HandSolder
- R49, R50, R51, R52, R53, R54, R58: footprint bca-footprints:R_L3.6mm_D1.6mm_P5.00mm_Horizontal -> Resistor_SMD:R_0603_1608Metric_Pad0.98x0.95mm_HandSolder
- R55: value 1k -> 330R; footprint bca-footprints:R_L3.6mm_D1.6mm_P5.00mm_Horizontal -> Resistor_SMD:R_0603_1608Metric_Pad0.98x0.95mm_HandSolder
- R56: value 2k -> 1k; footprint bca-footprints:R_L3.6mm_D1.6mm_P5.00mm_Horizontal -> Resistor_SMD:R_0603_1608Metric_Pad0.98x0.95mm_HandSolder
- R57: value 12k -> 2k; footprint bca-footprints:R_L3.6mm_D1.6mm_P5.00mm_Horizontal -> Resistor_SMD:R_0603_1608Metric_Pad0.98x0.95mm_HandSolder
- R59: value 3.3k -> 12k; footprint bca-footprints:R_L3.6mm_D1.6mm_P5.00mm_Horizontal -> Resistor_SMD:R_0603_1608Metric_Pad0.98x0.95mm_HandSolder
- R6: value 220k -> 470R
- R60: value 33k -> 3.3k; footprint bca-footprints:R_L3.6mm_D1.6mm_P5.00mm_Horizontal -> Resistor_SMD:R_0603_1608Metric_Pad0.98x0.95mm_HandSolder
- R61: value 470R -> 39k
- R62: value 330R -> 39k
- SW2: value SW_SPDT -> SW_DPDT_x2; footprint bca-footprints:SW_Toggle_SPDT_SolderLug -> bca-footprints:Pin_Header_Straight_1x06_Pitch2.54mm
- U1: value TLV9302 -> TLV9352
- U4: value TLV9301 -> TLV9351
- moved C35 146.6 mm to (96.5, -18.1)
- moved C42 144.4 mm to (102.2, -4.17)
- moved C31 144.3 mm to (96.5, -25.6)
- moved C34 142.3 mm to (96.5, -21.8)
- moved C29 142.2 mm to (96.5, -33.0)
- moved C30 142.1 mm to (96.5, -29.3)
- moved C41 141.5 mm to (102.2, -6.68)
- moved R41 140.1 mm to (88.6, -7.92)
- moved R42 139.4 mm to (88.6, -5.08)
- moved R39 139.3 mm to (88.6, -13.6)
- moved C33 139.3 mm to (96.0, 4.55)
- moved R40 139.2 mm to (88.6, -10.8)
- moved R43 138.6 mm to (88.6, -2.25)
- moved R46 138.5 mm to (88.6, 6.28)
- moved R45 138.2 mm to (88.6, 3.44)
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- renumbered SW3 to SWe
Connections:
- C13 pad 1: Net-(C13-Pad1) -> Earth
- C13 pad 2: +15V -> Net-(Q3-S)
- C14 pad 1: Net-(C14-Pad1) -> Net-(Q3-D)
- C14 pad 2: Net-(C13-Pad1) -> +15V
- C15 pad 1: Earth -> Net-(C15-Pad1)
- C15 pad 2: /Signal Path/ccs3 -> Net-(Q3-D)
- C16 pad 1: Net-(C16-Pad1) -> Earth
- C16 pad 2: +15V -> Net-(Q4-G)
- C17 pad 1: Net-(C17-Pad1) -> Earth
- C17 pad 2: Net-(C16-Pad1) -> /Signal Path/ccs3
- C18 pad 1: /Signal Path/eq_send -> Net-(Q4-D)
- C18 pad 2: Net-(C18-Pad2) -> +15V
- C19 pad 1: Earth -> Net-(C19-Pad1)
- C19 pad 2: Net-(C19-Pad2) -> Net-(Q4-D)
- C20 pad 1: Net-(C20-Pad1) -> /Signal Path/eq_send
- C20 pad 2: Net-(C20-Pad2) -> Net-(Q5-E)
- C21 pad 1: Net-(C20-Pad2) -> Earth
- C21 pad 2: Net-(C21-Pad2) -> Net-(U3B-+)
- C22 pad 2: Net-(C22-Pad2) -> Net-(U1B-+)
- C23 pad 1: Net-(C22-Pad2) -> Net-(C23-Pad1)
- C24 pad 1: Net-(C24-Pad1) -> Net-(C23-Pad2)
- C24 pad 2: Net-(C24-Pad2) -> Net-(U1A-+)
- C25 pad 1: Net-(C24-Pad2) -> Net-(C25-Pad1)
- C26 pad 1: Net-(C26-Pad1) -> Net-(U3B--)
- C28 pad 1: Net-(C28-Pad1) -> Net-(Q6A-D1)
- C28 pad 2: Net-(C28-Pad2) -> Net-(Q6B-D2)
- C29 pad 2: Net-(C28-Pad1) -> Net-(Q6A-D1)
- C30 pad 2: Net-(C28-Pad2) -> Net-(Q6B-D2)
- C31 pad 2: Net-(C31-Pad2) -> Net-(Q6B-G1)
- C36 pad 1: Net-(C36-Pad1) -> Net-(C35-Pad2)
- C36 pad 2: Net-(C35-Pad2) -> Net-(C36-Pad2)
- C37 pad 2: Earth -> Net-(C35-Pad2)
- C38 pad 2: Net-(C38-Pad2) -> Net-(U4A-+)
- C47 pad 1: +15V -> Net-(D3-K)
- C48 pad 1: Earth -> Net-(D3-K)
- C48 pad 2: -15V -> Earth
- C7 pad 2: Net-(C7-Pad2) -> Net-(RV1A-6)
- C8 pad 1: Net-(C8-Pad1) -> Net-(Q2-G)
- D3 pad 1: Net-(C37-Pad1) -> Net-(D3-K)
- D4 pad 1: Net-(C37-Pad1) -> Net-(D3-K)
- J1 pad 3: Net-(J1-Pad3) -> unconnected-(J1-Pad3)
- J4 pad 4: Net-(C37-Pad1) -> /return
- J4 pad 5: +15V -> /output_jack
- J4 pad 8: -15V -> unconnected-(J4-Pin_8-Pad8)
- J5 pad 4: /return -> Net-(D3-K)
- J5 pad 5: /output_jack -> +15V
- J5 pad 8: Net-(J5-Pad8) -> -15V
- Q1 pad 2: Net-(Q1-Pad2) -> Net-(Q1-S)
- Q10 pad 2: Net-(Q10-Pad2) -> Net-(Q10-E)
- Q11 pad 2: Net-(Q11-Pad2) -> Net-(Q11-E)
- Q12 pad 2: Net-(Q12-Pad2) -> Net-(Q12-E)
- Q13 pad 2: Net-(Q13-Pad2) -> Net-(Q13-E)
- Q2 pad 3: Net-(Q2-Pad3) -> Net-(Q2-G)
- Q3 pad 1: Net-(C13-Pad1) -> Net-(Q3-D)
- Q3 pad 2: Net-(C12-Pad2) -> Net-(Q3-S)
- Q3 pad 3: Net-(Q3-Pad3) -> Net-(Q3-G)
- Q4 pad 1: Net-(C16-Pad1) -> Net-(Q4-D)
- Q4 pad 2: Net-(Q4-Pad2) -> Net-(Q4-S)
- Q4 pad 3: Net-(Q4-Pad3) -> Net-(Q4-G)
- Q5 pad 1: Net-(Q5-Pad1) -> Net-(Q5-B)
- Q5 pad 2: Net-(C18-Pad2) -> Net-(Q5-E)
- Q6 pad 1: Net-(Q6-Pad1) -> Net-(Q6A-G1)
- Q6 pad 2: Net-(C28-Pad1) -> Net-(Q6A-D1)
- Q6 pad 4: Net-(C31-Pad2) -> Net-(Q6B-G1)
- Q6 pad 5: Net-(C28-Pad2) -> Net-(Q6B-D2)
- Q7 pad 2: Net-(Q7-Pad2) -> Net-(Q7-E)
- Q7 pad 3: Net-(Q7-Pad3) -> Net-(Q7-C)
- Q8 pad 1: Net-(Q7-Pad3) -> Net-(Q7-C)
- Q9 pad 2: Net-(Q9-Pad2) -> Net-(Q9-E)
- R12 pad 2: Net-(R12-Pad2) -> Net-(C12-Pad2)
- R13 pad 1: Net-(R12-Pad2) -> Net-(C12-Pad2)
- R15 pad 1: Net-(R15-Pad1) -> +15V
- R15 pad 2: Net-(Q3-Pad3) -> Net-(Q3-D)
- R16 pad 1: +15V -> Net-(Q3-S)
- R16 pad 2: Net-(C13-Pad1) -> /Signal Path/ccs2
- R17 pad 1: Net-(C12-Pad2) -> Net-(C15-Pad1)
- R17 pad 2: /Signal Path/ccs2 -> Net-(Q4-G)
- R18 pad 1: Net-(C14-Pad1) -> Net-(Q4-G)
- R18 pad 2: Net-(R18-Pad2) -> /Signal Path/-VREF0
- R19 pad 1: Net-(R18-Pad2) -> +15V
- R19 pad 2: /Signal Path/-VREF0 -> Net-(Q4-D)
- R20 pad 1: Net-(R18-Pad2) -> Net-(Q4-S)
- R20 pad 2: Net-(Q4-Pad3) -> /Signal Path/ccs3
- R21 pad 1: +15V -> Net-(C19-Pad1)
- R21 pad 2: Net-(C16-Pad1) -> Net-(Q5-B)
- R22 pad 1: Net-(Q4-Pad2) -> Net-(Q5-B)
- R22 pad 2: /Signal Path/ccs3 -> Earth
- R23 pad 1: Net-(C17-Pad1) -> Net-(Q5-E)
- R23 pad 2: Net-(Q5-Pad1) -> -15V
- R24 pad 1: Net-(Q5-Pad1) -> /Signal Path/eq_send
- R24 pad 2: Earth -> Net-(U3B-+)
- R25 pad 1: Net-(C18-Pad2) -> Net-(U3B-+)
- R25 pad 2: -15V -> Earth
- R26 pad 1: Net-(C20-Pad2) -> Net-(C22-Pad1)
- R27 pad 1: /Signal Path/eq_send -> Net-(U1B-+)
- R27 pad 2: Net-(C19-Pad2) -> Earth
- R28 pad 1: Net-(C21-Pad2) -> Net-(C23-Pad2)
- R28 pad 2: Earth -> Net-(U1A--)
- R29 pad 1: Net-(C22-Pad2) -> Net-(U1A-+)
- R29 pad 2: Net-(R29-Pad2) -> Earth
- R30 pad 1: Net-(C23-Pad2) -> Net-(C25-Pad2)
- R31 pad 1: Net-(C24-Pad2) -> Net-(C26-Pad2)
- R31 pad 2: Net-(R31-Pad2) -> Net-(U3B--)
- R32 pad 1: Net-(C25-Pad2) -> Net-(C27-Pad1)
- R32 pad 2: Earth -> /Signal Path/-VREF1
- R33 pad 1: Net-(C26-Pad2) -> Net-(C27-Pad1)
- R33 pad 2: Net-(C26-Pad1) -> Net-(Q6A-G1)
- R34 pad 1: Net-(C27-Pad1) -> +15V
- R34 pad 2: /Signal Path/-VREF1 -> Net-(Q6A-D1)
- R35 pad 1: Net-(C27-Pad1) -> +15V
- R35 pad 2: Net-(Q6-Pad1) -> Net-(Q6B-D2)
- R36 pad 1: +15V -> Net-(Q6B-G1)
- R36 pad 2: Net-(C28-Pad1) -> /Signal Path/-VREF1
- R37 pad 1: +15V -> Net-(C29-Pad1)
- R37 pad 2: Net-(C28-Pad2) -> Net-(C32-Pad2)
- R38 pad 1: Net-(C31-Pad2) -> Net-(C30-Pad1)
- R38 pad 2: /Signal Path/-VREF1 -> Net-(C33-Pad2)
- R39 pad 1: Net-(C29-Pad1) -> Net-(C31-Pad1)
- R39 pad 2: Net-(C32-Pad2) -> Earth
- R40 pad 1: Net-(C30-Pad1) -> Net-(C33-Pad2)
- R40 pad 2: Net-(C33-Pad2) -> Earth
- R41 pad 2: Earth -> Net-(C34-Pad1)
- R42 pad 1: Net-(C31-Pad1) -> Net-(C32-Pad2)
- R42 pad 2: Net-(C34-Pad1) -> Net-(U3A--)
- R43 pad 2: Earth -> Net-(U3A-+)
- R44 pad 1: Net-(C32-Pad2) -> Net-(C31-Pad1)
- R44 pad 2: Net-(R44-Pad2) -> Net-(C36-Pad2)
- R45 pad 1: Net-(C33-Pad2) -> Net-(C32-Pad2)
- R45 pad 2: Net-(R45-Pad2) -> Net-(C35-Pad2)
- R46 pad 1: Net-(C32-Pad2) -> Net-(C31-Pad1)
- R47 pad 1: Net-(C31-Pad1) -> Earth
- R47 pad 2: Net-(C35-Pad2) -> Net-(Q7-C)
- R48 pad 1: Earth -> Net-(Q7-E)
- R48 pad 2: Net-(Q7-Pad3) -> -15V
- R49 pad 1: Net-(Q7-Pad2) -> Net-(Q9-E)
- R5 pad 1: Net-(Q1-Pad2) -> Net-(Q1-S)
- R50 pad 1: Net-(Q9-Pad2) -> Net-(Q10-E)
- R51 pad 1: Net-(Q10-Pad2) -> Net-(Q11-E)
- R52 pad 1: Net-(Q11-Pad2) -> Net-(Q12-E)
- R53 pad 1: Net-(Q12-Pad2) -> Net-(Q12-E)
- R54 pad 1: Net-(Q13-Pad2) -> Net-(Q13-E)
- R55 pad 1: Earth -> Net-(Q13-E)
- R55 pad 2: Net-(C38-Pad2) -> -15V
- R56 pad 1: Net-(C38-Pad2) -> Earth
- R56 pad 2: Net-(R56-Pad2) -> Net-(U4A-+)
- R57 pad 1: Net-(R56-Pad2) -> Net-(U4A-+)
- R57 pad 2: -15V -> Net-(R57-Pad2)
- R58 pad 1: Earth -> Net-(R57-Pad2)
- R58 pad 2: /Signal Path/-VREF1 -> -15V
- R59 pad 1: /Signal Path/-VREF1 -> Earth
- R59 pad 2: -15V -> /Signal Path/-VREF1
- R6 pad 1: Net-(C4-Pad1) -> Net-(Q1-S)
- R6 pad 2: Net-(C7-Pad2) -> Net-(SW2A-A)
- R60 pad 1: +15V -> /Signal Path/-VREF1
- R60 pad 2: /V+ -> -15V
- R61 pad 1: Net-(Q12-Pad2) -> +15V
- R61 pad 2: -15V -> /V+
- R62 pad 1: Net-(Q13-Pad2) -> +15V
- R62 pad 2: -15V -> Net-(D6-A1)
- R7 pad 1: Net-(C7-Pad2) -> Net-(C4-Pad1)
- R7 pad 2: /Signal Path/-VREF0 -> Net-(RV1A-6)
- R8 pad 1: Net-(R8-Pad1) -> Net-(RV1A-6)
- R9 pad 1: Net-(C8-Pad1) -> Net-(RV1A-4)
- R9 pad 2: Net-(Q2-Pad3) -> /Signal Path/-VREF0
- RV1 pad 1: Net-(R8-Pad1) -> Net-(RV1A-4)
- RV1 pad 2: Net-(C8-Pad1) -> Net-(Q2-G)
- RV1 pad 3: Net-(C7-Pad2) -> Net-(RV1A-6)
- RV1 pad 5: Net-(R15-Pad1) -> Net-(Q3-G)
- RV1 pad 6: Net-(R12-Pad2) -> Net-(C12-Pad2)
- RV2 pad 1: Net-(C19-Pad2) -> Net-(U3B-+)
- RV2 pad 2: Net-(C20-Pad1) -> Net-(C22-Pad1)
- RV2 pad 3: Net-(C26-Pad1) -> Net-(U3B--)
- RV3 pad 1: Net-(C19-Pad2) -> Net-(U3B-+)
- RV3 pad 2: Net-(C22-Pad1) -> Net-(C23-Pad1)
- RV3 pad 3: Net-(C26-Pad1) -> Net-(U3B--)
- RV4 pad 1: Net-(C19-Pad2) -> Net-(U3B-+)
- RV4 pad 2: Net-(C24-Pad1) -> Net-(C25-Pad1)
- RV4 pad 3: Net-(C26-Pad1) -> Net-(U3B--)
- RV5 pad 3: Net-(C36-Pad1) -> Net-(C37-Pad1)
- SW1 pad 3: Net-(SW1-Pad3) -> unconnected-(SW1A-C-Pad3)
- SW1 pad 6: Net-(SW1-Pad6) -> unconnected-(SW1B-C-Pad6)
- SW2 pad 1: Net-(Q1-Pad2) -> Net-(SW2A-A)
- SWe pad 2: Net-(C7-Pad2) -> Net-(RV1A-6)
- SWe pad 3: Net-(SW3-Pad3) -> unconnected-(SW3-C-Pad3)
- U1 pad 1: Net-(R29-Pad2) -> Net-(U1A--)
- U1 pad 2: Net-(R29-Pad2) -> Net-(U1A--)
- U1 pad 3: Net-(C23-Pad2) -> Net-(U1A-+)
- U1 pad 5: Net-(C21-Pad2) -> Net-(U1B-+)
- U3 pad 2: Net-(R44-Pad2) -> Net-(U3A--)
- U3 pad 3: Net-(R45-Pad2) -> Net-(U3A-+)
- U3 pad 5: Net-(C19-Pad2) -> Net-(U3B-+)
- U3 pad 6: Net-(C26-Pad1) -> Net-(U3B--)
- U4 pad 3: Net-(C38-Pad2) -> Net-(U4A-+)
Routing:
- net /input_jack: track 190.2 -> 0.00 mm
- net /return: track 168.1 -> 0.00 mm
- net /Signal Path/-VREF0: track 138.2 -> 0.00 mm, vias 2 -> 0
- net /LED+: track 120.5 -> 0.00 mm
- net Net-(C19-Pad2): track 99.5 -> 0.00 mm
- net Earth: track 96.7 -> 0.00 mm, vias 12 -> 0
- net /Signal Path/ccs0: track 94.9 -> 0.00 mm, vias 2 -> 0
- net Net-(C37-Pad1): track 83.5 -> 0.00 mm, vias 1 -> 0
- net /output_jack: track 77.5 -> 0.00 mm
- net Net-(C26-Pad1): track 71.5 -> 0.00 mm
- net Net-(C7-Pad2): track 70.5 -> 0.00 mm
- net Net-(R15-Pad1): track 67.2 -> 0.00 mm
- net Net-(C8-Pad1): track 63.3 -> 0.00 mm
- net Net-(R12-Pad2): track 60.3 -> 0.00 mm
- net Net-(Q1-Pad2): track 59.1 -> 0.00 mm, vias 1 -> 0
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- removed copper zone on In2.Cu, net +15V
- removed copper zone on In2.Cu, net -15V
- removed copper zone on F.Cu, net /Signal Path/-VREF1
- removed copper zone on F.Cu, net Earth
- removed copper zone on F.Cu, net Net-(C37-Pad1)
- removed copper zone on F.Cu, net Net-(C38-Pad2)
- removed copper zone on F.Cu, net Net-(D1-K)
- removed copper zone on F.Cu, net Net-(D2-K)
Other:
- outline, holes or cut-outs redrawn
- net class Default removed
- board text added: "BCA Sea Eagle v1.1.0; Feb 2024"
- board text removed: "BCA Distortion v1.0.0; Dec 2023"

Commit message: first draft of PCB
Parts:
- moved C44 98.5 mm to (3.80, -17.8)
- moved C43 96.6 mm to (3.80, -24.8)
- moved C17 95.6 mm to (13.1, -0.68)
- moved R24 93.4 mm to (21.7, 9.97), turned to 0 degrees
- moved U1 91.9 mm to (3.80, -21.3)
- moved R23 90.4 mm to (12.9, 9.96)
- moved R28 90.4 mm to (-5.00, -17.1)
- moved R29 90.1 mm to (-5.00, -15.0)
- moved R30 89.8 mm to (-5.00, -12.9), turned to 0 degrees
- moved R25 89.2 mm to (21.7, 7.45)
- moved R22 89.0 mm to (12.9, 15.0), turned to 0 degrees
- moved R21 89.0 mm to (12.9, 12.5), turned to 180 degrees
- moved C15 84.8 mm to (12.9, -4.90), turned to 180 degrees
- moved C28 84.8 mm to (21.6, -30.0)
- moved C20 84.1 mm to (12.9, 6.97)
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- renumbered SWe to SW3
Connections:
- C21 pad 2: Net-(U3B-+) -> Net-(U3A-+)
- C26 pad 1: Net-(U3B--) -> Net-(U3A--)
- R24 pad 2: Net-(U3B-+) -> Net-(U3A-+)
- R25 pad 1: Net-(U3B-+) -> Net-(U3A-+)
- R31 pad 2: Net-(U3B--) -> Net-(U3A--)
- R42 pad 2: Net-(U3A--) -> Net-(U3B--)
- R43 pad 2: Net-(U3A-+) -> Net-(U3B-+)
- RV2 pad 1: Net-(U3B-+) -> Net-(U3A-+)
- RV2 pad 3: Net-(U3B--) -> Net-(U3A--)
- RV3 pad 1: Net-(U3B-+) -> Net-(U3A-+)
- RV3 pad 3: Net-(U3B--) -> Net-(U3A--)
- RV4 pad 1: Net-(U3B-+) -> Net-(U3A-+)
- RV4 pad 3: Net-(U3B--) -> Net-(U3A--)
- SW2 pad 3: /Signal Path/ccs0 -> Net-(Q1-S)
- U3 pad 1: Net-(C35-Pad2) -> Net-(C26-Pad2)
- U3 pad 7: Net-(C26-Pad2) -> Net-(C35-Pad2)
Routing:
- net +15V: track 0.00 -> 242.5 mm, vias 0 -> 9
- net -15V: track 0.00 -> 218.3 mm, vias 0 -> 5
- net /input_jack: track 0.00 -> 194.0 mm
- net /Signal Path/-VREF0: track 0.00 -> 118.5 mm, vias 0 -> 2
- net /send: track 0.00 -> 109.0 mm
- net Earth: track 0.00 -> 96.4 mm, vias 0 -> 20
- net Net-(U3A-+): track 0.00 -> 86.7 mm
- net Net-(D3-K): track 0.00 -> 77.7 mm, vias 0 -> 1
- net /output_jack: track 0.00 -> 73.6 mm
- net Net-(U3A--): track 0.00 -> 71.5 mm
- net Net-(Q1-S): track 0.00 -> 65.9 mm
- net /Signal Path/ccs4: track 0.00 -> 61.1 mm, vias 0 -> 2
- net Net-(C12-Pad2): track 0.00 -> 60.8 mm
- net Net-(C31-Pad1): track 0.00 -> 60.1 mm
- net Net-(Q3-G): track 0.00 -> 55.9 mm
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- added copper zone on F.Cu, net Earth
- added copper zone on F.Cu, net Net-(D1-K)
- added copper zone on F.Cu, net Net-(D2-K)
- added copper zone on F.Cu, net Net-(D3-K)
Other:
- board text added: "ALL 20kW POTS USE CENTER DETENT"
- board text removed: "ALL 100kB POTS USE CENTER DETENT"
- board text removed: "LTP"
- board text removed: "Q1"
- board text removed: "Q2"
- board text removed: "Q3"
- board text removed: "Q4"
