File: tight-distortion.kicad_pcb (KiCad board)
At the start: 4 copper layers, 110 x 84.3 mm, 147 parts, among them J1 Barrel_Jack_Switch, J2 AudioJack_TRS, J3 AudioJack_TRS, J4 Conn_01x08, J5 power-module, Q1 MMBFJ202, Q10 BC848C, Q11 BC848C, Q12 BC848C, Q13 BC848C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

Commit message: small schematic change
Connections:
- R62 pad 2: Net-(D6-A1) -> Net-(D6-A2)
- SW2 pad 6: Net-(D6-A2) -> Net-(D6-A1)
Routing:
- net Net-(D6-A1): track 24.6 -> 8.61 mm
- net Net-(D6-A2): track 15.1 -> 29.7 mm
Other:
- board text removed: "ALL SWITCHES ON-ON"
Changed lines of the file:
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@@
     (property "ki_keywords" "switch dual-pole double-throw DPDT spdt ON-ON")
     (attr through_hole)
-    (fp_text reference "SW2" (at 0 -2.5 180) (layer "F.SilkS") hide
+    (fp_text reference "SW2" (at 9.4 0 180) (layer "F.SilkS")
         (effects (font (size 1 1) (thickness 0.15)))
     )
@@
       (net 90 "Net-(SW2B-B)") (pinfunction "B") (pintype "passive"))
     (pad "6" thru_hole oval locked (at 6.35 0 90) (size 1.7 1.7) (drill 1) (layers "*.Cu" "*.Mask")
-      (net 94 "Net-(D6-A2)") (pinfunction "C") (pintype "passive"))
+      (net 67 "Net-(D6-A1)") (pinfunction "C") (pintype "passive"))
     (model "${KISYS3DMOD}/Pin_Headers.3dshapes/Pin_Header_Straight_1x06_Pitch2.54mm.wrl"
       (offset (xyz 0 0 0))
@@
       (net 10 "+15V") (pintype "passive"))
     (pad "2" thru_hole oval (at 2.5 0) (size 1.4 1.4) (drill 0.7) (layers "*.Cu" "*.Mask")
-      (net 67 "Net-(D6-A1)") (pintype "passive"))
+      (net 94 "Net-(D6-A2)") (pintype "passive"))
     (model "${KISYS3DMOD}/Resistors_THT.3dshapes/R_Axial_DIN0204_L3.6mm_D1.6mm_P5.08mm_Horizontal.wrl"
       (offset (xyz 0 0 0))
@@
     (effects (font (size 1 1) (thickness 0.15)) (justify mirror))
   )
-  (gr_text "ALL SWITCHES ON-ON" (at -37.4 14.6) (layer "B.SilkS")
-    (effects (font (size 1 1) (thickness 0.15)) (justify mirror))
-  )
   (gr_text "Designed & Assembled \nin St. John's, NL" (at 38 -13.4) (layer "F.SilkS")
     (effects (font (size 1 1) (thickness 0.15)))
@@
   (segment (start -21.652651 -38.8) (end -21.652651 -38.302651) (width 1) (layer "B.Cu") (net 64))
   (segment (start -21.652651 -38.302651) (end -15.775 -32.425) (width 1) (layer "B.Cu") (net 64))
-  (segment (start -45.75 14.15) (end -47.5 12.4) (width 0.25) (layer "F.Cu") (net 67))
-  (segment (start -38.85 14.15) (end -45.75 14.15) (width 0.25) (layer "F.Cu") (net 67))
-  (segment (start -26.64 15.9) (end -37.1 15.9) (width 0.25) (layer "F.Cu") (net 67))
-  (segment (start -25.04 17.5) (end -26.64 15.9) (width 0.25) (layer "F.Cu") (net 67))
-  (segment (start -37.1 15.9) (end -38.85 14.15) (width 0.25) (layer "F.Cu") (net 67))
+  (segment (start -33.65 17.5) (end -25.04 17.5) (width 0.25) (layer "F.Cu") (net 67))
   (segment (start -33.6 7.5) (end -29.2 7.5) (width 0.25) (layer "F.Cu") (net 70))
   (segment (start -47.5 10.2) (end -46 8.7) (width 0.25) (layer "F.Cu") (net 70))
@@
   (segment (start -39.09 14.6) (end -36.19 17.5) (width 0.25) (layer "F.Cu") (net 90))
   (segment (start -47.5 14.6) (end -39.09 14.6) (width 0.25) (layer "F.Cu") (net 90))
-  (segment (start -21.66 19.2) (end -19.96 17.5) (width 0.25) (layer "F.Cu") (net 94))
-  (segment (start -31.95 19.2) (end -21.66 19.2) (width 0.25) (layer "F.Cu") (net 94))
-  (segment (start -33.65 17.5) (end -31.95 19.2) (width 0.25) (layer "F.Cu") (net 94))
+  (segment (start -21.56 15.9) (end -37.153604 15.9) (width 0.25) (layer "F.Cu") (net 94))
+  (segment (start -37.153604 15.9) (end -38.903604 14.15) (width 0.25) (layer "F.Cu") (net 94))
+  (segment (start -45.75 14.15) (end -47.5 12.4) (width 0.25) (layer "F.Cu") (net 94))
+  (segment (start -19.96 17.5) (end -21.56 15.9) (width 0.25) (layer "F.Cu") (net 94))
+  (segment (start -38.903604 14.15) (end -45.75 14.15) (width 0.25) (layer "F.Cu") (net 94))
   (zone (net 1) (net_name "Earth") (layer "F.Cu") (hatch edge 0.5)
     (priority 3)

Commit message: final look at PCB
Parts:
- SW1, SW3: moved to B.Cu
- moved C4 0.55 mm to (-41.6, -3.70)
- moved C2 0.55 mm to (-41.6, 4.30)
- moved C8 0.55 mm to (-44.9, 4.30)
- moved J4 0.50 mm to (40.0, 17.0)
- moved SW2 0.50 mm to (-40.0, 17.0)
- turned SW1 to 0 degrees
- turned SW3 to 180 degrees
Routing:
- net +15V: track 242.5 -> 37.9 mm
- net -15V: track 218.3 -> 18.3 mm, vias 5 -> 13
- net Net-(Q1-D): track 30.1 -> 36.5 mm
- net Net-(SW1B-B): track 41.2 -> 35.2 mm
- net Net-(SW1B-A): track 7.20 -> 12.4 mm
- net /return: track 45.5 -> 50.1 mm, vias 1 -> 0
- net Net-(C31-Pad1): track 60.1 -> 62.4 mm
- net /input_jack: track 194.0 -> 196.0 mm
- net Net-(C29-Pad1): track 21.7 -> 23.5 mm
- net Net-(C30-Pad1): track 24.0 -> 25.9 mm
- net Net-(Q2-G): track 43.2 -> 44.2 mm
- net Net-(U3A-+): track 86.7 -> 87.4 mm
- net Net-(SW2A-A): track 11.6 -> 11.0 mm
- net /output_jack: track 73.6 -> 73.0 mm
- net Net-(SW2A-B): track 17.8 -> 17.2 mm
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- added copper zone on In2.Cu, net +15V
- added copper zone on In2.Cu, net -15V
Other:
- board text added: "Bennett Custom Audio Sea Eagle Distortion v1.1.0; Feb 2024"
- board text removed: "BCA Sea Eagle v1.1.0; Feb 2024"
